File: vmc/pcb/mdb_interface.kicad_sch (KiCad schematic)
At the start: 29 parts, among them J10 ONE_WIRE_1, J11 ONE_WIRE_2, J12 AUX_1, J13 AUX_2, J14 AUX_3, J4 MDB_CONN, J9 PICO_DEBUG_HEADER, Q14 BC817, Q15 MMBT3906, Q16 BSS138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

Commit message: Add resistor values
Parts:
- R38: value R -> 1K4
- R39, R40, R41: value R -> 60R4
Changed lines of the file:
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@@
 			)
 		)
-		(property "Value" "R"
+		(property "Value" "1K4"
 			(at 39.37 177.8 90)
 			(effects
@@
 			)
 		)
-		(property "Value" "R"
+		(property "Value" "60R4"
 			(at 146.05 177.8 90)
 			(effects
@@
 			)
 		)
-		(property "Value" "R"
+		(property "Value" "60R4"
 			(at 109.22 177.8 90)
 			(effects
@@
 			)
 		)
-		(property "Value" "R"
+		(property "Value" "60R4"
 			(at 68.58 177.8 90)
 			(effects

Commit message: Add version number to PCB (v1.1) Whitespace formatting
Parts:
- R37: value 700R -> 750R
- R38: value 1K4 -> 1.4K
- R39, R40, R41: value 60R4 -> 5.1R
Changed lines of the file:
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@@
 			)
 		)
-		(property "Value" "1K4"
+		(property "Value" "1.4K"
 			(at 39.37 177.8 90)
 			(effects
@@
 			)
 		)
-		(property "Value" "60R4"
+		(property "Value" "5.1R"
 			(at 146.05 177.8 90)
 			(effects
@@
 			)
 		)
-		(property "Value" "700R"
+		(property "Value" "750R"
 			(at 25.4 92.456 0)
 			(effects
@@
 			)
 		)
-		(property "Value" "60R4"
+		(property "Value" "5.1R"
 			(at 109.22 177.8 90)
 			(effects
@@
 			)
 		)
-		(property "Value" "60R4"
+		(property "Value" "5.1R"
 			(at 68.58 177.8 90)
 			(effects

Commit message: Update 5R to 5R1
Parts:
- R29: value 5R -> 5R1
Changed lines of the file:
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@@
 			)
 		)
-		(property "Value" "5R"
+		(property "Value" "5R1"
 			(at 86.36 34.2899 0)
 			(effects

Commit message: Update schematic to use correct 60R4 resistor values Update stock info
Parts:
- R39, R40, R41: value 5.1R -> 60R4
Changed lines of the file:
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@@
 			)
 		)
-		(property "Value" "5.1R"
+		(property "Value" "60R4"
 			(at 146.05 177.8 90)
 			(effects
@@
 			)
 		)
-		(property "Value" "5.1R"
+		(property "Value" "60R4"
 			(at 109.22 177.8 90)
 			(effects
@@
 			)
 		)
-		(property "Value" "5.1R"
+		(property "Value" "60R4"
 			(at 68.58 177.8 90)
 			(effects
